Commit message: [Edit] Edit Joint name

File: urdf/robonex.urdf (robot description, URDF)
Before this commit: robot robonex, 25 links, 24 joints
Joints:
- removed joint l_ankle_actuator_joint_a
- removed joint l_ankle_actuator_joint_b
- removed joint l_ankle_foot_joint
- removed joint l_ankle_joint
- removed joint l_knee_actuator_joint
- removed joint r_ankle_actuator_joint_a
- removed joint r_ankle_actuator_joint_b
- removed joint r_ankle_foot_joint
- removed joint r_ankle_joint
- removed joint r_knee_actuator_joint
- added joint l_ankle_lower_joint: type revolute, parent l_knee_link, child l_ankle_crank_link_b, origin xyz=0.000000 0.002100 -0.255500 rpy=0 0 0, axis 0 1 0, limit lower=-3.141593 upper=3.141593 effort=17.0 velocity=42.9
- added joint l_ankle_pitch_joint: type revolute, parent l_ankle_link, child l_foot, origin xyz=-0.020000 -0.020000 -0.050000 rpy=0 0 0, axis 0 -1 0, limit lower=-3.141593 upper=3.141593 effort=0.0 velocity=0.0
- added joint l_ankle_roll_joint: type revolute, parent l_knee_link, child l_ankle_link, origin xyz=0.020000 0.025000 -0.326500 rpy=0 0 0, axis 1 0 0, limit lower=-3.141593 upper=3.141593 effort=0.0 velocity=0.0
- added joint l_ankle_upper_joint: type revolute, parent l_knee_link, child l_ankle_crank_link_a, origin xyz=0.000000 0.047900 -0.144500 rpy=0 0 0, axis 0 -1 0, limit lower=-3.141593 upper=3.141593 effort=17.0 velocity=42.9
- added joint l_knee_pitch_joint: type revolute, parent l_hip_roll_link, child l_knee_crank_link, origin xyz=-0.034800 -0.032000 -0.255000 rpy=0 0 0, axis 0 -1 0, limit lower=-0.872665 upper=0.087266 effort=60.0 velocity=20.9
- added joint r_ankle_lower_joint: type revolute, parent r_knee_link, child r_ankle_crank_link_a, origin xyz=0.000000 -0.002100 -0.255500 rpy=0 0 0, axis 0 -1 0, limit lower=-3.141593 upper=3.141593 effort=17.0 velocity=42.9
- added joint r_ankle_pitch_joint: type revolute, parent r_ankle_link, child r_foot, origin xyz=-0.020000 -0.021500 -0.050000 rpy=0 0 0, axis 0 -1 0, limit lower=-3.141593 upper=3.141593 effort=0.0 velocity=0.0
- added joint r_ankle_roll_joint: type revolute, parent r_knee_link, child r_ankle_link, origin xyz=0.020000 -0.025000 -0.326500 rpy=0 0 0, axis 1 0 0, limit lower=-3.141593 upper=3.141593 effort=0.0 velocity=0.0
- added joint r_ankle_upper_joint: type revolute, parent r_knee_link, child r_ankle_crank_link_b, origin xyz=0.000000 -0.047900 -0.144500 rpy=0 0 0, axis 0 1 0, limit lower=-3.141593 upper=3.141593 effort=17.0 velocity=42.9
- added joint r_knee_pitch_joint: type revolute, parent r_hip_roll_link, child r_knee_crank_link, origin xyz=-0.034800 0.032000 -0.255000 rpy=0 0 0, axis 0 1 0, limit lower=-0.087266 upper=0.872665 effort=60.0 velocity=20.9
- joint l_hip_pitch_joint: limit lower=-3.141593 upper=3.141593 effort=60.0 velocity=20.9 -> lower=-0.872665 upper=0.872665 effort=60.0 velocity=20.9
- joint l_hip_roll_joint: axis 1 0 0 -> -1 0 0; limit lower=-3.141593 upper=3.141593 effort=60.0 velocity=20.9 -> lower=-1.047198 upper=0.087266 effort=60.0 velocity=20.9
- joint l_hip_yaw_joint: limit lower=-3.141593 upper=3.141593 effort=17.0 velocity=42.9 -> lower=-0.698132 upper=0.698132 effort=17.0 velocity=42.9
- joint r_hip_pitch_joint: axis 0 -1 0 -> 0 1 0; limit lower=-3.141593 upper=3.141593 effort=60.0 velocity=20.9 -> lower=-0.872665 upper=0.872665 effort=60.0 velocity=20.9
- joint r_hip_roll_joint: axis 1 0 0 -> -1 0 0; limit lower=-3.141593 upper=3.141593 effort=60.0 velocity=20.9 -> lower=-0.087266 upper=1.047198 effort=60.0 velocity=20.9
- joint r_hip_yaw_joint: limit lower=-3.141593 upper=3.141593 effort=17.0 velocity=42.9 -> lower=-0.698132 upper=0.698132 effort=17.0 velocity=42.9
