Commit message: [Edit] Edit Isaac Model

File: ros2/robonex.urdf.xacro (robot description, xacro)
@@ -1,4 +1,3 @@
 <?xml version="1.0"?>
-<!-- generated by ros2/build_ros_urdf.py - do not edit by hand -->
 <robot name="robonex" xmlns:xacro="http://www.ros.org/wiki/xacro">
   <material name="black"><color rgba="0.05 0.05 0.05 1.0"/></material>
@@ -496,5 +495,5 @@
     <axis xyz="0 0 1"/>
     <limit lower="-0.698132" upper="0.698132" effort="17" velocity="42.9"/>
-    <dynamics damping="0.2" friction="0.0"/>
+    <dynamics damping="0.2" friction="0.1"/>
   </joint>
   <joint name="r_hip_yaw_joint" type="revolute">
@@ -504,5 +503,5 @@
     <axis xyz="0 0 1"/>
     <limit lower="-0.698132" upper="0.698132" effort="17" velocity="42.9"/>
-    <dynamics damping="0.2" friction="0.0"/>
+    <dynamics damping="0.2" friction="0.1"/>
   </joint>
   <joint name="l_hip_pitch_joint" type="revolute">
@@ -512,5 +511,5 @@
     <axis xyz="0 -1 0"/>
     <limit lower="-0.872665" upper="0.872665" effort="60" velocity="20.9"/>
-    <dynamics damping="0.2" friction="0.0"/>
+    <dynamics damping="0.2" friction="0.2"/>
   </joint>
   <joint name="r_hip_pitch_joint" type="revolute">
@@ -520,5 +519,5 @@
     <axis xyz="0 1 0"/>
     <limit lower="-0.872665" upper="0.872665" effort="60" velocity="20.9"/>
-    <dynamics damping="0.2" friction="0.0"/>
+    <dynamics damping="0.2" friction="0.2"/>
   </joint>
   <joint name="l_hip_roll_joint" type="revolute">
@@ -528,5 +527,5 @@
     <axis xyz="-1 0 0"/>
     <limit lower="-1.047198" upper="0.087266" effort="60" velocity="20.9"/>
-    <dynamics damping="0.2" friction="0.0"/>
+    <dynamics damping="0.2" friction="0.2"/>
   </joint>
   <joint name="r_hip_roll_joint" type="revolute">
@@ -536,5 +535,5 @@
     <axis xyz="-1 0 0"/>
     <limit lower="-0.087266" upper="1.047198" effort="60" velocity="20.9"/>
-    <dynamics damping="0.2" friction="0.0"/>
+    <dynamics damping="0.2" friction="0.2"/>
   </joint>
   <joint name="l_knee_joint" type="revolute">
@@ -544,5 +543,5 @@
     <axis xyz="0 -1 0"/>
     <limit lower="-0.733038" upper="0.059341" effort="85.1" velocity="14.7"/>
-    <dynamics damping="0.2" friction="0.0"/>
+    <dynamics damping="0.2" friction="0.284"/>
   </joint>
   <joint name="r_knee_joint" type="revolute">
@@ -552,5 +551,5 @@
     <axis xyz="0 1 0"/>
     <limit lower="-0.059341" upper="0.733038" effort="85.1" velocity="14.7"/>
-    <dynamics damping="0.2" friction="0.0"/>
+    <dynamics damping="0.2" friction="0.284"/>
   </joint>
   <joint name="l_knee_pitch_joint" type="fixed">
@@ -619,6 +618,6 @@
     <origin xyz="0.02 0.025 -0.3265" rpy="0 0 0"/>
     <axis xyz="1 0 0"/>
-    <limit lower="-0.272271" upper="0.258309" effort="33.5" velocity="43.5"/>
-    <dynamics damping="0.2" friction="0.0"/>
+    <limit lower="-0.253073" upper="0.244346" effort="33.5" velocity="43.5"/>
+    <dynamics damping="0.2" friction="0.198"/>
   </joint>
   <joint name="r_ankle_roll_joint" type="revolute">
@@ -627,6 +626,6 @@
     <origin xyz="0.02 -0.025 -0.3265" rpy="0 0 0"/>
     <axis xyz="1 0 0"/>
-    <limit lower="-0.258309" upper="0.272271" effort="33.5" velocity="43.5"/>
-    <dynamics damping="0.2" friction="0.0"/>
+    <limit lower="-0.235619" upper="0.244346" effort="33.5" velocity="43.5"/>
+    <dynamics damping="0.2" friction="0.198"/>
   </joint>
   <joint name="l_ankle_pitch_joint" type="revolute">
@@ -635,6 +634,6 @@
     <origin xyz="-0.02 -0.02 -0.05" rpy="0 0 0"/>
     <axis xyz="0 -1 0"/>
-    <limit lower="-0.336849" upper="0.284489" effort="34" velocity="42.9"/>
-    <dynamics damping="0.2" friction="0.0"/>
+    <limit lower="-0.357792" upper="0.279253" effort="34" velocity="42.9"/>
+    <dynamics damping="0.2" friction="0.2"/>
   </joint>
   <joint name="r_ankle_pitch_joint" type="revolute">
@@ -643,6 +642,6 @@
     <origin xyz="-0.02 -0.0215 -0.05" rpy="0 0 0"/>
     <axis xyz="0 -1 0"/>
-    <limit lower="-0.336849" upper="0.284489" effort="34" velocity="42.9"/>
-    <dynamics damping="0.2" friction="0.0"/>
+    <limit lower="-0.331613" upper="0.270526" effort="34" velocity="42.9"/>
+    <dynamics damping="0.2" friction="0.2"/>
   </joint>
   <ros2_control name="RoboNexSystem" type="system">
@@ -798,5 +797,5 @@
   </gazebo>
   <gazebo reference="l_foot">
-    <mu1>1</mu1><mu2>1</mu2>
+    <mu1>0.6</mu1><mu2>0.6</mu2>
     <self_collide>true</self_collide>
     <sensor name="l_foot_contact" type="contact">
@@ -808,5 +807,5 @@
   </gazebo>
   <gazebo reference="r_foot">
-    <mu1>1</mu1><mu2>1</mu2>
+    <mu1>0.6</mu1><mu2>0.6</mu2>
     <self_collide>true</self_collide>
     <sensor name="r_foot_contact" type="contact">

File: urdf/robonex.urdf (robot description, URDF)
Before this commit: robot robonex, 25 links, 24 joints
Joints:
- joint l_ankle_lower_joint: limit lower=-3.141593 upper=3.141593 effort=17.0 velocity=42.9 -> lower=-0.436332 upper=0.610865 effort=17.0 velocity=42.9
- joint l_ankle_upper_joint: limit lower=-3.141593 upper=3.141593 effort=17.0 velocity=42.9 -> lower=-0.610865 upper=0.436332 effort=17.0 velocity=42.9
- joint r_ankle_lower_joint: limit lower=-3.141593 upper=3.141593 effort=17.0 velocity=42.9 -> lower=-0.321141 upper=0.314159 effort=17.0 velocity=42.9
- joint r_ankle_upper_joint: limit lower=-3.141593 upper=3.141593 effort=17.0 velocity=42.9 -> lower=-0.289725 upper=0.296706 effort=17.0 velocity=42.9
