Commit message: [Edit] save

File: isaac/closed_loop_box/robonex_closed_loop_box.urdf (robot description, URDF)
Before this commit: robot robonex, 25 links, 24 joints
Joints:
- joint r_ankle_lower_joint: limit lower=-0.321141 upper=0.314159 effort=17 velocity=42.9 -> lower=-0.610865 upper=0.436332 effort=17 velocity=42.9
- joint r_ankle_upper_joint: limit lower=-0.289725 upper=0.296706 effort=17 velocity=42.9 -> lower=-0.436332 upper=0.610865 effort=17 velocity=42.9

File: isaac/closed_loop_mesh/robonex_closed_loop_mesh.urdf (robot description, URDF)
Before this commit: robot robonex, 25 links, 24 joints
Joints:
- joint r_ankle_lower_joint: limit lower=-0.321141 upper=0.314159 effort=17 velocity=42.9 -> lower=-0.610865 upper=0.436332 effort=17 velocity=42.9
- joint r_ankle_upper_joint: limit lower=-0.289725 upper=0.296706 effort=17 velocity=42.9 -> lower=-0.436332 upper=0.610865 effort=17 velocity=42.9

File: urdf/robonex.urdf (robot description, URDF)
Before this commit: robot robonex, 25 links, 24 joints
Joints:
- joint r_ankle_lower_joint: limit lower=-0.321141 upper=0.314159 effort=17.0 velocity=42.9 -> lower=-0.610865 upper=0.436332 effort=17.0 velocity=42.9
- joint r_ankle_upper_joint: limit lower=-0.289725 upper=0.296706 effort=17.0 velocity=42.9 -> lower=-0.436332 upper=0.610865 effort=17.0 velocity=42.9

Commit message: [Fix] Free the ankle rod-end bolt axis in both Isaac and MuJoCo

File: isaac/closed_loop_box/robonex_closed_loop_box.urdf (robot description, URDF)
Before this commit: robot robonex, 25 links, 24 joints
Joints:
- joint l_ankle_pitch_joint: limit lower=-3.141593 upper=3.141593 effort=0 velocity=0 -> effort=0 velocity=0; type revolute -> continuous
- joint l_ankle_roll_joint: limit lower=-3.141593 upper=3.141593 effort=0 velocity=0 -> effort=0 velocity=0; type revolute -> continuous
- joint l_knee_coupler_joint_a: limit lower=-3.141593 upper=3.141593 effort=0 velocity=0 -> effort=0 velocity=0; type revolute -> continuous
- joint l_knee_joint: limit lower=-3.141593 upper=3.141593 effort=0 velocity=0 -> effort=0 velocity=0; type revolute -> continuous
- joint r_ankle_pitch_joint: limit lower=-3.141593 upper=3.141593 effort=0 velocity=0 -> effort=0 velocity=0; type revolute -> continuous
- joint r_ankle_roll_joint: limit lower=-3.141593 upper=3.141593 effort=0 velocity=0 -> effort=0 velocity=0; type revolute -> continuous
- joint r_knee_coupler_joint_a: limit lower=-3.141593 upper=3.141593 effort=0 velocity=0 -> effort=0 velocity=0; type revolute -> continuous
- joint r_knee_joint: limit lower=-3.141593 upper=3.141593 effort=0 velocity=0 -> effort=0 velocity=0; type revolute -> continuous

File: isaac/closed_loop_mesh/robonex_closed_loop_mesh.urdf (robot description, URDF)
Before this commit: robot robonex, 25 links, 24 joints
Joints:
- joint l_ankle_pitch_joint: limit lower=-3.141593 upper=3.141593 effort=0 velocity=0 -> effort=0 velocity=0; type revolute -> continuous
- joint l_ankle_roll_joint: limit lower=-3.141593 upper=3.141593 effort=0 velocity=0 -> effort=0 velocity=0; type revolute -> continuous
- joint l_knee_coupler_joint_a: limit lower=-3.141593 upper=3.141593 effort=0 velocity=0 -> effort=0 velocity=0; type revolute -> continuous
- joint l_knee_joint: limit lower=-3.141593 upper=3.141593 effort=0 velocity=0 -> effort=0 velocity=0; type revolute -> continuous
- joint r_ankle_pitch_joint: limit lower=-3.141593 upper=3.141593 effort=0 velocity=0 -> effort=0 velocity=0; type revolute -> continuous
- joint r_ankle_roll_joint: limit lower=-3.141593 upper=3.141593 effort=0 velocity=0 -> effort=0 velocity=0; type revolute -> continuous
- joint r_knee_coupler_joint_a: limit lower=-3.141593 upper=3.141593 effort=0 velocity=0 -> effort=0 velocity=0; type revolute -> continuous
- joint r_knee_joint: limit lower=-3.141593 upper=3.141593 effort=0 velocity=0 -> effort=0 velocity=0; type revolute -> continuous

Commit message: [Edit] robot limit

File: isaac/closed_loop_box/robonex_closed_loop_box.urdf (robot description, URDF)
Before this commit: robot robonex, 25 links, 24 joints
Joints:
- joint l_ankle_lower_joint: limit lower=-0.436332 upper=0.610865 effort=17 velocity=42.9 -> lower=-0.610865 upper=0.575959 effort=17 velocity=42.9
- joint l_ankle_upper_joint: limit lower=-0.610865 upper=0.436332 effort=17 velocity=42.9 -> lower=-0.610865 upper=0.575959 effort=17 velocity=42.9
- joint l_hip_pitch_joint: limit lower=-0.872665 upper=0.872665 effort=60 velocity=20.9 -> lower=-1.745329 upper=1.745329 effort=60 velocity=20.9
- joint l_hip_roll_joint: limit lower=-1.047198 upper=0.087266 effort=60 velocity=20.9 -> lower=-2.146755 upper=0.453786 effort=60 velocity=20.9
- joint l_hip_yaw_joint: limit lower=-0.698132 upper=0.698132 effort=17 velocity=42.9 -> lower=-1.658063 upper=1.658063 effort=17 velocity=42.9
- joint l_knee_pitch_joint: limit lower=-0.872665 upper=0.087266 effort=60 velocity=20.9 -> lower=-1.500983 upper=0.942478 effort=60 velocity=20.9
- joint r_ankle_lower_joint: limit lower=-0.610865 upper=0.436332 effort=17 velocity=42.9 -> lower=-0.575959 upper=0.610865 effort=17 velocity=42.9
- joint r_ankle_upper_joint: limit lower=-0.436332 upper=0.610865 effort=17 velocity=42.9 -> lower=-0.575959 upper=0.610865 effort=17 velocity=42.9
- joint r_hip_pitch_joint: limit lower=-0.872665 upper=0.872665 effort=60 velocity=20.9 -> lower=-1.745329 upper=1.745329 effort=60 velocity=20.9
- joint r_hip_roll_joint: limit lower=-0.087266 upper=1.047198 effort=60 velocity=20.9 -> lower=-0.453786 upper=2.146755 effort=60 velocity=20.9
- joint r_hip_yaw_joint: limit lower=-0.698132 upper=0.698132 effort=17 velocity=42.9 -> lower=-1.658063 upper=1.658063 effort=17 velocity=42.9
- joint r_knee_pitch_joint: limit lower=-0.087266 upper=0.872665 effort=60 velocity=20.9 -> lower=-0.942478 upper=1.500983 effort=60 velocity=20.9

File: isaac/closed_loop_mesh/robonex_closed_loop_mesh.urdf (robot description, URDF)
Before this commit: robot robonex, 25 links, 24 joints
Joints:
- joint l_ankle_lower_joint: limit lower=-0.436332 upper=0.610865 effort=17 velocity=42.9 -> lower=-0.610865 upper=0.575959 effort=17 velocity=42.9
- joint l_ankle_upper_joint: limit lower=-0.610865 upper=0.436332 effort=17 velocity=42.9 -> lower=-0.610865 upper=0.575959 effort=17 velocity=42.9
- joint l_hip_pitch_joint: limit lower=-0.872665 upper=0.872665 effort=60 velocity=20.9 -> lower=-1.745329 upper=1.745329 effort=60 velocity=20.9
- joint l_hip_roll_joint: limit lower=-1.047198 upper=0.087266 effort=60 velocity=20.9 -> lower=-2.146755 upper=0.453786 effort=60 velocity=20.9
- joint l_hip_yaw_joint: limit lower=-0.698132 upper=0.698132 effort=17 velocity=42.9 -> lower=-1.658063 upper=1.658063 effort=17 velocity=42.9
- joint l_knee_pitch_joint: limit lower=-0.872665 upper=0.087266 effort=60 velocity=20.9 -> lower=-1.500983 upper=0.942478 effort=60 velocity=20.9
- joint r_ankle_lower_joint: limit lower=-0.610865 upper=0.436332 effort=17 velocity=42.9 -> lower=-0.575959 upper=0.610865 effort=17 velocity=42.9
- joint r_ankle_upper_joint: limit lower=-0.436332 upper=0.610865 effort=17 velocity=42.9 -> lower=-0.575959 upper=0.610865 effort=17 velocity=42.9
- joint r_hip_pitch_joint: limit lower=-0.872665 upper=0.872665 effort=60 velocity=20.9 -> lower=-1.745329 upper=1.745329 effort=60 velocity=20.9
- joint r_hip_roll_joint: limit lower=-0.087266 upper=1.047198 effort=60 velocity=20.9 -> lower=-0.453786 upper=2.146755 effort=60 velocity=20.9
- joint r_hip_yaw_joint: limit lower=-0.698132 upper=0.698132 effort=17 velocity=42.9 -> lower=-1.658063 upper=1.658063 effort=17 velocity=42.9
- joint r_knee_pitch_joint: limit lower=-0.087266 upper=0.872665 effort=60 velocity=20.9 -> lower=-0.942478 upper=1.500983 effort=60 velocity=20.9

File: ros2/robonex.urdf.xacro (robot description, xacro)
@@ -494,5 +494,5 @@
     <origin xyz="0.060424 0.05 -0.20245" rpy="0 0 0"/>
     <axis xyz="0 0 1"/>
-    <limit lower="-0.698132" upper="0.698132" effort="17" velocity="42.9"/>
+    <limit lower="-1.658063" upper="1.658063" effort="17" velocity="42.9"/>
     <dynamics damping="0.2" friction="0.1"/>
   </joint>
@@ -502,5 +502,5 @@
     <origin xyz="0.060424 -0.05 -0.20245" rpy="0 0 0"/>
     <axis xyz="0 0 1"/>
-    <limit lower="-0.698132" upper="0.698132" effort="17" velocity="42.9"/>
+    <limit lower="-1.658063" upper="1.658063" effort="17" velocity="42.9"/>
     <dynamics damping="0.2" friction="0.1"/>
   </joint>
@@ -510,5 +510,5 @@
     <origin xyz="1e-06 0.0477 -0.0605" rpy="0 0 0"/>
     <axis xyz="0 -1 0"/>
-    <limit lower="-0.872665" upper="0.872665" effort="60" velocity="20.9"/>
+    <limit lower="-1.745329" upper="1.745329" effort="60" velocity="20.9"/>
     <dynamics damping="0.2" friction="0.2"/>
   </joint>
@@ -518,5 +518,5 @@
     <origin xyz="-1e-06 -0.0477 -0.0605" rpy="0 0 0"/>
     <axis xyz="0 1 0"/>
-    <limit lower="-0.872665" upper="0.872665" effort="60" velocity="20.9"/>
+    <limit lower="-1.745329" upper="1.745329" effort="60" velocity="20.9"/>
     <dynamics damping="0.2" friction="0.2"/>
   </joint>
@@ -526,5 +526,5 @@
     <origin xyz="0.0225 0.0623 -0.034" rpy="0 0 0"/>
     <axis xyz="-1 0 0"/>
-    <limit lower="-1.047198" upper="0.087266" effort="60" velocity="20.9"/>
+    <limit lower="-2.146755" upper="0.453786" effort="60" velocity="20.9"/>
     <dynamics damping="0.2" friction="0.2"/>
   </joint>
@@ -534,5 +534,5 @@
     <origin xyz="0.0225 -0.0627 -0.034" rpy="0 0 0"/>
     <axis xyz="-1 0 0"/>
-    <limit lower="-0.087266" upper="1.047198" effort="60" velocity="20.9"/>
+    <limit lower="-0.453786" upper="2.146755" effort="60" velocity="20.9"/>
     <dynamics damping="0.2" friction="0.2"/>
   </joint>
@@ -542,5 +542,5 @@
     <origin xyz="-0.0348 -0.0255 -0.34" rpy="0 0 0"/>
     <axis xyz="0 -1 0"/>
-    <limit lower="-0.733038" upper="0.059341" effort="85.1" velocity="14.7"/>
+    <limit lower="-1.242674" upper="0.485202" effort="85.1" velocity="14.7"/>
     <dynamics damping="0.2" friction="0.284"/>
   </joint>
@@ -550,5 +550,5 @@
     <origin xyz="-0.0348 0.0255 -0.34" rpy="0 0 0"/>
     <axis xyz="0 1 0"/>
-    <limit lower="-0.059341" upper="0.733038" effort="85.1" velocity="14.7"/>
+    <limit lower="-0.485202" upper="1.242674" effort="85.1" velocity="14.7"/>
     <dynamics damping="0.2" friction="0.284"/>
   </joint>
@@ -618,5 +618,5 @@
     <origin xyz="0.02 0.025 -0.3265" rpy="0 0 0"/>
     <axis xyz="1 0 0"/>
-    <limit lower="-0.253073" upper="0.244346" effort="33.5" velocity="43.5"/>
+    <limit lower="-0.520108" upper="0.427606" effort="33.5" velocity="43.5"/>
     <dynamics damping="0.2" friction="0.198"/>
   </joint>
@@ -626,5 +626,5 @@
     <origin xyz="0.02 -0.025 -0.3265" rpy="0 0 0"/>
     <axis xyz="1 0 0"/>
-    <limit lower="-0.235619" upper="0.244346" effort="33.5" velocity="43.5"/>
+    <limit lower="-0.427606" upper="0.520108" effort="33.5" velocity="43.5"/>
     <dynamics damping="0.2" friction="0.198"/>
   </joint>
@@ -634,5 +634,5 @@
     <origin xyz="-0.02 -0.02 -0.05" rpy="0 0 0"/>
     <axis xyz="0 -1 0"/>
-    <limit lower="-0.357792" upper="0.279253" effort="34" velocity="42.9"/>
+    <limit lower="-0.729548" upper="0.520108" effort="34" velocity="42.9"/>
     <dynamics damping="0.2" friction="0.2"/>
   </joint>
@@ -642,5 +642,5 @@
     <origin xyz="-0.02 -0.0215 -0.05" rpy="0 0 0"/>
     <axis xyz="0 -1 0"/>
-    <limit lower="-0.331613" upper="0.270526" effort="34" velocity="42.9"/>
+    <limit lower="-0.729548" upper="0.520108" effort="34" velocity="42.9"/>
     <dynamics damping="0.2" friction="0.2"/>
   </joint>

File: urdf/robonex.urdf (robot description, URDF)
Before this commit: robot robonex, 25 links, 24 joints
Joints:
- joint l_ankle_lower_joint: limit lower=-0.436332 upper=0.610865 effort=17.0 velocity=42.9 -> lower=-0.610865 upper=0.575959 effort=17.0 velocity=42.9
- joint l_ankle_upper_joint: limit lower=-0.610865 upper=0.436332 effort=17.0 velocity=42.9 -> lower=-0.610865 upper=0.575959 effort=17.0 velocity=42.9
- joint l_hip_pitch_joint: limit lower=-0.872665 upper=0.872665 effort=60.0 velocity=20.9 -> lower=-1.745329 upper=1.745329 effort=60.0 velocity=20.9
- joint l_hip_roll_joint: limit lower=-1.047198 upper=0.087266 effort=60.0 velocity=20.9 -> lower=-2.146755 upper=0.453786 effort=60.0 velocity=20.9
- joint l_hip_yaw_joint: limit lower=-0.698132 upper=0.698132 effort=17.0 velocity=42.9 -> lower=-1.658063 upper=1.658063 effort=17.0 velocity=42.9
- joint l_knee_pitch_joint: limit lower=-0.872665 upper=0.087266 effort=60.0 velocity=20.9 -> lower=-1.500983 upper=0.942478 effort=60.0 velocity=20.9
- joint r_ankle_lower_joint: limit lower=-0.610865 upper=0.436332 effort=17.0 velocity=42.9 -> lower=-0.575959 upper=0.610865 effort=17.0 velocity=42.9
- joint r_ankle_upper_joint: limit lower=-0.436332 upper=0.610865 effort=17.0 velocity=42.9 -> lower=-0.575959 upper=0.610865 effort=17.0 velocity=42.9
- joint r_hip_pitch_joint: limit lower=-0.872665 upper=0.872665 effort=60.0 velocity=20.9 -> lower=-1.745329 upper=1.745329 effort=60.0 velocity=20.9
- joint r_hip_roll_joint: limit lower=-0.087266 upper=1.047198 effort=60.0 velocity=20.9 -> lower=-0.453786 upper=2.146755 effort=60.0 velocity=20.9
- joint r_hip_yaw_joint: limit lower=-0.698132 upper=0.698132 effort=17.0 velocity=42.9 -> lower=-1.658063 upper=1.658063 effort=17.0 velocity=42.9
- joint r_knee_pitch_joint: limit lower=-0.087266 upper=0.872665 effort=60.0 velocity=20.9 -> lower=-0.942478 upper=1.500983 effort=60.0 velocity=20.9
