Commit message: [Edit] Ver.2 hip limits from the user (yaw 90, pitch 100, roll -120..10); degree-based limit tool

File: new_urdf/isaac/edu/closed_loop_box/robonex_edu_closed_loop_box.urdf (robot description, URDF)
Before this commit: robot robonex_edu, 25 links, 24 joints
Joints:
- joint l_hip_roll_joint: limit lower=-2.146755 upper=0.453786 effort=60 velocity=20.9 -> lower=-2.094395 upper=0.174533 effort=60 velocity=20.9
- joint l_hip_yaw_joint: limit lower=-1.658063 upper=1.658063 effort=17 velocity=42.9 -> lower=-1.570796 upper=1.570796 effort=17 velocity=42.9
- joint r_hip_roll_joint: limit lower=-0.453786 upper=2.146755 effort=60 velocity=20.9 -> lower=-0.174533 upper=2.094395 effort=60 velocity=20.9
- joint r_hip_yaw_joint: limit lower=-1.658063 upper=1.658063 effort=17 velocity=42.9 -> lower=-1.570796 upper=1.570796 effort=17 velocity=42.9

File: new_urdf/isaac/edu/closed_loop_mesh/robonex_edu_closed_loop_mesh.urdf (robot description, URDF)
Before this commit: robot robonex_edu, 25 links, 24 joints
Joints:
- joint l_hip_roll_joint: limit lower=-2.146755 upper=0.453786 effort=60 velocity=20.9 -> lower=-2.094395 upper=0.174533 effort=60 velocity=20.9
- joint l_hip_yaw_joint: limit lower=-1.658063 upper=1.658063 effort=17 velocity=42.9 -> lower=-1.570796 upper=1.570796 effort=17 velocity=42.9
- joint r_hip_roll_joint: limit lower=-0.453786 upper=2.146755 effort=60 velocity=20.9 -> lower=-0.174533 upper=2.094395 effort=60 velocity=20.9
- joint r_hip_yaw_joint: limit lower=-1.658063 upper=1.658063 effort=17 velocity=42.9 -> lower=-1.570796 upper=1.570796 effort=17 velocity=42.9

File: new_urdf/isaac/max/closed_loop_box/robonex_max_closed_loop_box.urdf (robot description, URDF)
Before this commit: robot robonex_max, 34 links, 33 joints
Joints:
- joint l_hip_roll_joint: limit lower=-2.146755 upper=0.453786 effort=60 velocity=20.9 -> lower=-2.094395 upper=0.174533 effort=60 velocity=20.9
- joint l_hip_yaw_joint: limit lower=-1.658063 upper=1.658063 effort=17 velocity=42.9 -> lower=-1.570796 upper=1.570796 effort=17 velocity=42.9
- joint r_hip_roll_joint: limit lower=-0.453786 upper=2.146755 effort=60 velocity=20.9 -> lower=-0.174533 upper=2.094395 effort=60 velocity=20.9
- joint r_hip_yaw_joint: limit lower=-1.658063 upper=1.658063 effort=17 velocity=42.9 -> lower=-1.570796 upper=1.570796 effort=17 velocity=42.9

File: new_urdf/isaac/max/closed_loop_mesh/robonex_max_closed_loop_mesh.urdf (robot description, URDF)
Before this commit: robot robonex_max, 34 links, 33 joints
Joints:
- joint l_hip_roll_joint: limit lower=-2.146755 upper=0.453786 effort=60 velocity=20.9 -> lower=-2.094395 upper=0.174533 effort=60 velocity=20.9
- joint l_hip_yaw_joint: limit lower=-1.658063 upper=1.658063 effort=17 velocity=42.9 -> lower=-1.570796 upper=1.570796 effort=17 velocity=42.9
- joint r_hip_roll_joint: limit lower=-0.453786 upper=2.146755 effort=60 velocity=20.9 -> lower=-0.174533 upper=2.094395 effort=60 velocity=20.9
- joint r_hip_yaw_joint: limit lower=-1.658063 upper=1.658063 effort=17 velocity=42.9 -> lower=-1.570796 upper=1.570796 effort=17 velocity=42.9

File: new_urdf/isaac/pro/closed_loop_box/robonex_pro_closed_loop_box.urdf (robot description, URDF)
Before this commit: robot robonex_pro, 33 links, 32 joints
Joints:
- joint l_hip_roll_joint: limit lower=-2.146755 upper=0.453786 effort=60 velocity=20.9 -> lower=-2.094395 upper=0.174533 effort=60 velocity=20.9
- joint l_hip_yaw_joint: limit lower=-1.658063 upper=1.658063 effort=17 velocity=42.9 -> lower=-1.570796 upper=1.570796 effort=17 velocity=42.9
- joint r_hip_roll_joint: limit lower=-0.453786 upper=2.146755 effort=60 velocity=20.9 -> lower=-0.174533 upper=2.094395 effort=60 velocity=20.9
- joint r_hip_yaw_joint: limit lower=-1.658063 upper=1.658063 effort=17 velocity=42.9 -> lower=-1.570796 upper=1.570796 effort=17 velocity=42.9

File: new_urdf/isaac/pro/closed_loop_mesh/robonex_pro_closed_loop_mesh.urdf (robot description, URDF)
Before this commit: robot robonex_pro, 33 links, 32 joints
Joints:
- joint l_hip_roll_joint: limit lower=-2.146755 upper=0.453786 effort=60 velocity=20.9 -> lower=-2.094395 upper=0.174533 effort=60 velocity=20.9
- joint l_hip_yaw_joint: limit lower=-1.658063 upper=1.658063 effort=17 velocity=42.9 -> lower=-1.570796 upper=1.570796 effort=17 velocity=42.9
- joint r_hip_roll_joint: limit lower=-0.453786 upper=2.146755 effort=60 velocity=20.9 -> lower=-0.174533 upper=2.094395 effort=60 velocity=20.9
- joint r_hip_yaw_joint: limit lower=-1.658063 upper=1.658063 effort=17 velocity=42.9 -> lower=-1.570796 upper=1.570796 effort=17 velocity=42.9

File: new_urdf/urdf/robonex_edu.urdf (robot description, URDF)
Before this commit: robot robonex_edu, 25 links, 24 joints
Joints:
- joint l_hip_pitch_joint: limit lower=-3.141593 upper=3.141593 effort=60.0 velocity=20.9 -> lower=-1.745329 upper=1.745329 effort=60.0 velocity=20.9
- joint l_hip_roll_joint: limit lower=-3.141593 upper=3.141593 effort=60.0 velocity=20.9 -> lower=-2.094395 upper=0.174533 effort=60.0 velocity=20.9
- joint l_hip_yaw_joint: limit lower=-3.141593 upper=3.141593 effort=17.0 velocity=42.9 -> lower=-1.570796 upper=1.570796 effort=17.0 velocity=42.9
- joint r_hip_pitch_joint: limit lower=-3.141593 upper=3.141593 effort=60.0 velocity=20.9 -> lower=-1.745329 upper=1.745329 effort=60.0 velocity=20.9
- joint r_hip_roll_joint: limit lower=-3.141593 upper=3.141593 effort=60.0 velocity=20.9 -> lower=-0.174533 upper=2.094395 effort=60.0 velocity=20.9
- joint r_hip_yaw_joint: limit lower=-3.141593 upper=3.141593 effort=17.0 velocity=42.9 -> lower=-1.570796 upper=1.570796 effort=17.0 velocity=42.9

File: new_urdf/urdf/robonex_max.urdf (robot description, URDF)
Before this commit: robot robonex_max, 34 links, 33 joints
Joints:
- joint l_hip_pitch_joint: limit lower=-3.141593 upper=3.141593 effort=60.0 velocity=20.9 -> lower=-1.745329 upper=1.745329 effort=60.0 velocity=20.9
- joint l_hip_roll_joint: limit lower=-3.141593 upper=3.141593 effort=60.0 velocity=20.9 -> lower=-2.094395 upper=0.174533 effort=60.0 velocity=20.9
- joint l_hip_yaw_joint: limit lower=-3.141593 upper=3.141593 effort=17.0 velocity=42.9 -> lower=-1.570796 upper=1.570796 effort=17.0 velocity=42.9
- joint r_hip_pitch_joint: limit lower=-3.141593 upper=3.141593 effort=60.0 velocity=20.9 -> lower=-1.745329 upper=1.745329 effort=60.0 velocity=20.9
- joint r_hip_roll_joint: limit lower=-3.141593 upper=3.141593 effort=60.0 velocity=20.9 -> lower=-0.174533 upper=2.094395 effort=60.0 velocity=20.9
- joint r_hip_yaw_joint: limit lower=-3.141593 upper=3.141593 effort=17.0 velocity=42.9 -> lower=-1.570796 upper=1.570796 effort=17.0 velocity=42.9

File: new_urdf/urdf/robonex_pro.urdf (robot description, URDF)
Before this commit: robot robonex_pro, 33 links, 32 joints
Joints:
- joint l_hip_pitch_joint: limit lower=-3.141593 upper=3.141593 effort=60.0 velocity=20.9 -> lower=-1.745329 upper=1.745329 effort=60.0 velocity=20.9
- joint l_hip_roll_joint: limit lower=-3.141593 upper=3.141593 effort=60.0 velocity=20.9 -> lower=-2.094395 upper=0.174533 effort=60.0 velocity=20.9
- joint l_hip_yaw_joint: limit lower=-3.141593 upper=3.141593 effort=17.0 velocity=42.9 -> lower=-1.570796 upper=1.570796 effort=17.0 velocity=42.9
- joint r_hip_pitch_joint: limit lower=-3.141593 upper=3.141593 effort=60.0 velocity=20.9 -> lower=-1.745329 upper=1.745329 effort=60.0 velocity=20.9
- joint r_hip_roll_joint: limit lower=-3.141593 upper=3.141593 effort=60.0 velocity=20.9 -> lower=-0.174533 upper=2.094395 effort=60.0 velocity=20.9
- joint r_hip_yaw_joint: limit lower=-3.141593 upper=3.141593 effort=17.0 velocity=42.9 -> lower=-1.570796 upper=1.570796 effort=17.0 velocity=42.9

Commit message: [Edit] Ver.2 hip yaw limit +-48 deg (hip-yaw link meets the other leg's hip-pitch motor at 50)

File: new_urdf/isaac/edu/closed_loop_box/robonex_edu_closed_loop_box.urdf (robot description, URDF)
Before this commit: robot robonex_edu, 25 links, 24 joints
Joints:
- joint l_hip_yaw_joint: limit lower=-1.570796 upper=1.570796 effort=17 velocity=42.9 -> lower=-0.837758 upper=0.837758 effort=17 velocity=42.9
- joint r_hip_yaw_joint: limit lower=-1.570796 upper=1.570796 effort=17 velocity=42.9 -> lower=-0.837758 upper=0.837758 effort=17 velocity=42.9

File: new_urdf/isaac/edu/closed_loop_mesh/robonex_edu_closed_loop_mesh.urdf (robot description, URDF)
Before this commit: robot robonex_edu, 25 links, 24 joints
Joints:
- joint l_hip_yaw_joint: limit lower=-1.570796 upper=1.570796 effort=17 velocity=42.9 -> lower=-0.837758 upper=0.837758 effort=17 velocity=42.9
- joint r_hip_yaw_joint: limit lower=-1.570796 upper=1.570796 effort=17 velocity=42.9 -> lower=-0.837758 upper=0.837758 effort=17 velocity=42.9

File: new_urdf/isaac/max/closed_loop_box/robonex_max_closed_loop_box.urdf (robot description, URDF)
Before this commit: robot robonex_max, 34 links, 33 joints
Joints:
- joint l_hip_yaw_joint: limit lower=-1.570796 upper=1.570796 effort=17 velocity=42.9 -> lower=-0.837758 upper=0.837758 effort=17 velocity=42.9
- joint r_hip_yaw_joint: limit lower=-1.570796 upper=1.570796 effort=17 velocity=42.9 -> lower=-0.837758 upper=0.837758 effort=17 velocity=42.9

File: new_urdf/isaac/max/closed_loop_mesh/robonex_max_closed_loop_mesh.urdf (robot description, URDF)
Before this commit: robot robonex_max, 34 links, 33 joints
Joints:
- joint l_hip_yaw_joint: limit lower=-1.570796 upper=1.570796 effort=17 velocity=42.9 -> lower=-0.837758 upper=0.837758 effort=17 velocity=42.9
- joint r_hip_yaw_joint: limit lower=-1.570796 upper=1.570796 effort=17 velocity=42.9 -> lower=-0.837758 upper=0.837758 effort=17 velocity=42.9

File: new_urdf/isaac/pro/closed_loop_box/robonex_pro_closed_loop_box.urdf (robot description, URDF)
Before this commit: robot robonex_pro, 33 links, 32 joints
Joints:
- joint l_hip_yaw_joint: limit lower=-1.570796 upper=1.570796 effort=17 velocity=42.9 -> lower=-0.837758 upper=0.837758 effort=17 velocity=42.9
- joint r_hip_yaw_joint: limit lower=-1.570796 upper=1.570796 effort=17 velocity=42.9 -> lower=-0.837758 upper=0.837758 effort=17 velocity=42.9

File: new_urdf/isaac/pro/closed_loop_mesh/robonex_pro_closed_loop_mesh.urdf (robot description, URDF)
Before this commit: robot robonex_pro, 33 links, 32 joints
Joints:
- joint l_hip_yaw_joint: limit lower=-1.570796 upper=1.570796 effort=17 velocity=42.9 -> lower=-0.837758 upper=0.837758 effort=17 velocity=42.9
- joint r_hip_yaw_joint: limit lower=-1.570796 upper=1.570796 effort=17 velocity=42.9 -> lower=-0.837758 upper=0.837758 effort=17 velocity=42.9

File: new_urdf/urdf/robonex_edu.urdf (robot description, URDF)
Before this commit: robot robonex_edu, 25 links, 24 joints
Joints:
- joint l_hip_yaw_joint: limit lower=-1.570796 upper=1.570796 effort=17.0 velocity=42.9 -> lower=-0.837758 upper=0.837758 effort=17.0 velocity=42.9
- joint r_hip_yaw_joint: limit lower=-1.570796 upper=1.570796 effort=17.0 velocity=42.9 -> lower=-0.837758 upper=0.837758 effort=17.0 velocity=42.9

File: new_urdf/urdf/robonex_max.urdf (robot description, URDF)
Before this commit: robot robonex_max, 34 links, 33 joints
Joints:
- joint l_hip_yaw_joint: limit lower=-1.570796 upper=1.570796 effort=17.0 velocity=42.9 -> lower=-0.837758 upper=0.837758 effort=17.0 velocity=42.9
- joint r_hip_yaw_joint: limit lower=-1.570796 upper=1.570796 effort=17.0 velocity=42.9 -> lower=-0.837758 upper=0.837758 effort=17.0 velocity=42.9

File: new_urdf/urdf/robonex_pro.urdf (robot description, URDF)
Before this commit: robot robonex_pro, 33 links, 32 joints
Joints:
- joint l_hip_yaw_joint: limit lower=-1.570796 upper=1.570796 effort=17.0 velocity=42.9 -> lower=-0.837758 upper=0.837758 effort=17.0 velocity=42.9
- joint r_hip_yaw_joint: limit lower=-1.570796 upper=1.570796 effort=17.0 velocity=42.9 -> lower=-0.837758 upper=0.837758 effort=17.0 velocity=42.9
