Commit message: [Edit] Ver.2 hip pitch limit +-100 -> +-95 deg (CAD hip_roll_link-base_link contact from -96 backward)

File: ver2/isaac/edu/closed_loop_box/robonex_edu_closed_loop_box.urdf (robot description, URDF)
Before this commit: robot robonex_edu, 25 links, 24 joints
Joints:
- joint l_hip_pitch_joint: limit lower=-1.745329 upper=1.745329 effort=60 velocity=20.9 -> lower=-1.658063 upper=1.658063 effort=60 velocity=20.9
- joint r_hip_pitch_joint: limit lower=-1.745329 upper=1.745329 effort=60 velocity=20.9 -> lower=-1.658063 upper=1.658063 effort=60 velocity=20.9

File: ver2/isaac/edu/closed_loop_mesh/robonex_edu_closed_loop_mesh.urdf (robot description, URDF)
Before this commit: robot robonex_edu, 25 links, 24 joints
Joints:
- joint l_hip_pitch_joint: limit lower=-1.745329 upper=1.745329 effort=60 velocity=20.9 -> lower=-1.658063 upper=1.658063 effort=60 velocity=20.9
- joint r_hip_pitch_joint: limit lower=-1.745329 upper=1.745329 effort=60 velocity=20.9 -> lower=-1.658063 upper=1.658063 effort=60 velocity=20.9

File: ver2/isaac/max/closed_loop_box/robonex_max_closed_loop_box.urdf (robot description, URDF)
Before this commit: robot robonex_max, 34 links, 33 joints
Joints:
- joint l_hip_pitch_joint: limit lower=-1.745329 upper=1.745329 effort=60 velocity=20.9 -> lower=-1.658063 upper=1.658063 effort=60 velocity=20.9
- joint r_hip_pitch_joint: limit lower=-1.745329 upper=1.745329 effort=60 velocity=20.9 -> lower=-1.658063 upper=1.658063 effort=60 velocity=20.9

File: ver2/isaac/max/closed_loop_mesh/robonex_max_closed_loop_mesh.urdf (robot description, URDF)
Before this commit: robot robonex_max, 34 links, 33 joints
Joints:
- joint l_hip_pitch_joint: limit lower=-1.745329 upper=1.745329 effort=60 velocity=20.9 -> lower=-1.658063 upper=1.658063 effort=60 velocity=20.9
- joint r_hip_pitch_joint: limit lower=-1.745329 upper=1.745329 effort=60 velocity=20.9 -> lower=-1.658063 upper=1.658063 effort=60 velocity=20.9

File: ver2/isaac/pro/closed_loop_box/robonex_pro_closed_loop_box.urdf (robot description, URDF)
Before this commit: robot robonex_pro, 33 links, 32 joints
Joints:
- joint l_hip_pitch_joint: limit lower=-1.745329 upper=1.745329 effort=60 velocity=20.9 -> lower=-1.658063 upper=1.658063 effort=60 velocity=20.9
- joint r_hip_pitch_joint: limit lower=-1.745329 upper=1.745329 effort=60 velocity=20.9 -> lower=-1.658063 upper=1.658063 effort=60 velocity=20.9

File: ver2/isaac/pro/closed_loop_mesh/robonex_pro_closed_loop_mesh.urdf (robot description, URDF)
Before this commit: robot robonex_pro, 33 links, 32 joints
Joints:
- joint l_hip_pitch_joint: limit lower=-1.745329 upper=1.745329 effort=60 velocity=20.9 -> lower=-1.658063 upper=1.658063 effort=60 velocity=20.9
- joint r_hip_pitch_joint: limit lower=-1.745329 upper=1.745329 effort=60 velocity=20.9 -> lower=-1.658063 upper=1.658063 effort=60 velocity=20.9

File: ver2/urdf/robonex_edu.urdf (robot description, URDF)
Before this commit: robot robonex_edu, 25 links, 24 joints
Joints:
- joint l_hip_pitch_joint: limit lower=-1.745329 upper=1.745329 effort=60.0 velocity=20.9 -> lower=-1.658063 upper=1.658063 effort=60.0 velocity=20.9
- joint r_hip_pitch_joint: limit lower=-1.745329 upper=1.745329 effort=60.0 velocity=20.9 -> lower=-1.658063 upper=1.658063 effort=60.0 velocity=20.9

File: ver2/urdf/robonex_max.urdf (robot description, URDF)
Before this commit: robot robonex_max, 34 links, 33 joints
Joints:
- joint l_hip_pitch_joint: limit lower=-1.745329 upper=1.745329 effort=60.0 velocity=20.9 -> lower=-1.658063 upper=1.658063 effort=60.0 velocity=20.9
- joint r_hip_pitch_joint: limit lower=-1.745329 upper=1.745329 effort=60.0 velocity=20.9 -> lower=-1.658063 upper=1.658063 effort=60.0 velocity=20.9

File: ver2/urdf/robonex_pro.urdf (robot description, URDF)
Before this commit: robot robonex_pro, 33 links, 32 joints
Joints:
- joint l_hip_pitch_joint: limit lower=-1.745329 upper=1.745329 effort=60.0 velocity=20.9 -> lower=-1.658063 upper=1.658063 effort=60.0 velocity=20.9
- joint r_hip_pitch_joint: limit lower=-1.745329 upper=1.745329 effort=60.0 velocity=20.9 -> lower=-1.658063 upper=1.658063 effort=60.0 velocity=20.9

Commit message: [Edit] Ver.2 edu knee crank -70..+10, ankle upper -16..+50 / lower -50..+30 deg (left, mirrored right)

File: ver2/isaac/edu/closed_loop_box/robonex_edu_closed_loop_box.urdf (robot description, URDF)
Before this commit: robot robonex_edu, 25 links, 24 joints
Joints:
- joint l_ankle_lower_joint: limit lower=-0.610865 upper=0.575959 effort=17 velocity=42.9 -> lower=-0.872665 upper=0.523599 effort=17 velocity=42.9
- joint l_ankle_upper_joint: limit lower=-0.610865 upper=0.575959 effort=17 velocity=42.9 -> lower=-0.279253 upper=0.872665 effort=17 velocity=42.9
- joint l_knee_pitch_joint: limit lower=-1.361357 upper=0.261799 effort=60 velocity=20.9 -> lower=-1.221730 upper=0.174533 effort=60 velocity=20.9
- joint r_ankle_lower_joint: limit lower=-0.575959 upper=0.610865 effort=17 velocity=42.9 -> lower=-0.523599 upper=0.872665 effort=17 velocity=42.9
- joint r_ankle_upper_joint: limit lower=-0.575959 upper=0.610865 effort=17 velocity=42.9 -> lower=-0.872665 upper=0.279253 effort=17 velocity=42.9
- joint r_knee_pitch_joint: limit lower=-0.261799 upper=1.361357 effort=60 velocity=20.9 -> lower=-0.174533 upper=1.221730 effort=60 velocity=20.9

File: ver2/isaac/edu/closed_loop_mesh/robonex_edu_closed_loop_mesh.urdf (robot description, URDF)
Before this commit: robot robonex_edu, 25 links, 24 joints
Joints:
- joint l_ankle_lower_joint: limit lower=-0.610865 upper=0.575959 effort=17 velocity=42.9 -> lower=-0.872665 upper=0.523599 effort=17 velocity=42.9
- joint l_ankle_upper_joint: limit lower=-0.610865 upper=0.575959 effort=17 velocity=42.9 -> lower=-0.279253 upper=0.872665 effort=17 velocity=42.9
- joint l_knee_pitch_joint: limit lower=-1.361357 upper=0.261799 effort=60 velocity=20.9 -> lower=-1.221730 upper=0.174533 effort=60 velocity=20.9
- joint r_ankle_lower_joint: limit lower=-0.575959 upper=0.610865 effort=17 velocity=42.9 -> lower=-0.523599 upper=0.872665 effort=17 velocity=42.9
- joint r_ankle_upper_joint: limit lower=-0.575959 upper=0.610865 effort=17 velocity=42.9 -> lower=-0.872665 upper=0.279253 effort=17 velocity=42.9
- joint r_knee_pitch_joint: limit lower=-0.261799 upper=1.361357 effort=60 velocity=20.9 -> lower=-0.174533 upper=1.221730 effort=60 velocity=20.9

File: ver2/isaac/max/closed_loop_box/robonex_max_closed_loop_box.urdf (robot description, URDF)
Before this commit: robot robonex_max, 34 links, 33 joints
Joints:
- joint l_ankle_lower_joint: limit lower=-0.610865 upper=0.575959 effort=17 velocity=42.9 -> lower=-0.872665 upper=0.523599 effort=17 velocity=42.9
- joint l_ankle_upper_joint: limit lower=-0.610865 upper=0.575959 effort=17 velocity=42.9 -> lower=-0.279253 upper=0.872665 effort=17 velocity=42.9
- joint l_knee_pitch_joint: limit lower=-1.361357 upper=0.261799 effort=60 velocity=20.9 -> lower=-1.221730 upper=0.174533 effort=60 velocity=20.9
- joint r_ankle_lower_joint: limit lower=-0.575959 upper=0.610865 effort=17 velocity=42.9 -> lower=-0.523599 upper=0.872665 effort=17 velocity=42.9
- joint r_ankle_upper_joint: limit lower=-0.575959 upper=0.610865 effort=17 velocity=42.9 -> lower=-0.872665 upper=0.279253 effort=17 velocity=42.9
- joint r_knee_pitch_joint: limit lower=-0.261799 upper=1.361357 effort=60 velocity=20.9 -> lower=-0.174533 upper=1.221730 effort=60 velocity=20.9

File: ver2/isaac/max/closed_loop_mesh/robonex_max_closed_loop_mesh.urdf (robot description, URDF)
Before this commit: robot robonex_max, 34 links, 33 joints
Joints:
- joint l_ankle_lower_joint: limit lower=-0.610865 upper=0.575959 effort=17 velocity=42.9 -> lower=-0.872665 upper=0.523599 effort=17 velocity=42.9
- joint l_ankle_upper_joint: limit lower=-0.610865 upper=0.575959 effort=17 velocity=42.9 -> lower=-0.279253 upper=0.872665 effort=17 velocity=42.9
- joint l_knee_pitch_joint: limit lower=-1.361357 upper=0.261799 effort=60 velocity=20.9 -> lower=-1.221730 upper=0.174533 effort=60 velocity=20.9
- joint r_ankle_lower_joint: limit lower=-0.575959 upper=0.610865 effort=17 velocity=42.9 -> lower=-0.523599 upper=0.872665 effort=17 velocity=42.9
- joint r_ankle_upper_joint: limit lower=-0.575959 upper=0.610865 effort=17 velocity=42.9 -> lower=-0.872665 upper=0.279253 effort=17 velocity=42.9
- joint r_knee_pitch_joint: limit lower=-0.261799 upper=1.361357 effort=60 velocity=20.9 -> lower=-0.174533 upper=1.221730 effort=60 velocity=20.9

File: ver2/isaac/pro/closed_loop_box/robonex_pro_closed_loop_box.urdf (robot description, URDF)
Before this commit: robot robonex_pro, 33 links, 32 joints
Joints:
- joint l_ankle_lower_joint: limit lower=-0.610865 upper=0.575959 effort=17 velocity=42.9 -> lower=-0.872665 upper=0.523599 effort=17 velocity=42.9
- joint l_ankle_upper_joint: limit lower=-0.610865 upper=0.575959 effort=17 velocity=42.9 -> lower=-0.279253 upper=0.872665 effort=17 velocity=42.9
- joint l_knee_pitch_joint: limit lower=-1.361357 upper=0.261799 effort=60 velocity=20.9 -> lower=-1.221730 upper=0.174533 effort=60 velocity=20.9
- joint r_ankle_lower_joint: limit lower=-0.575959 upper=0.610865 effort=17 velocity=42.9 -> lower=-0.523599 upper=0.872665 effort=17 velocity=42.9
- joint r_ankle_upper_joint: limit lower=-0.575959 upper=0.610865 effort=17 velocity=42.9 -> lower=-0.872665 upper=0.279253 effort=17 velocity=42.9
- joint r_knee_pitch_joint: limit lower=-0.261799 upper=1.361357 effort=60 velocity=20.9 -> lower=-0.174533 upper=1.221730 effort=60 velocity=20.9

File: ver2/isaac/pro/closed_loop_mesh/robonex_pro_closed_loop_mesh.urdf (robot description, URDF)
Before this commit: robot robonex_pro, 33 links, 32 joints
Joints:
- joint l_ankle_lower_joint: limit lower=-0.610865 upper=0.575959 effort=17 velocity=42.9 -> lower=-0.872665 upper=0.523599 effort=17 velocity=42.9
- joint l_ankle_upper_joint: limit lower=-0.610865 upper=0.575959 effort=17 velocity=42.9 -> lower=-0.279253 upper=0.872665 effort=17 velocity=42.9
- joint l_knee_pitch_joint: limit lower=-1.361357 upper=0.261799 effort=60 velocity=20.9 -> lower=-1.221730 upper=0.174533 effort=60 velocity=20.9
- joint r_ankle_lower_joint: limit lower=-0.575959 upper=0.610865 effort=17 velocity=42.9 -> lower=-0.523599 upper=0.872665 effort=17 velocity=42.9
- joint r_ankle_upper_joint: limit lower=-0.575959 upper=0.610865 effort=17 velocity=42.9 -> lower=-0.872665 upper=0.279253 effort=17 velocity=42.9
- joint r_knee_pitch_joint: limit lower=-0.261799 upper=1.361357 effort=60 velocity=20.9 -> lower=-0.174533 upper=1.221730 effort=60 velocity=20.9
