Commit message: [Add] Ver.2 pro/max: arms and neck as actuated joints (common v1.2.0 placeholder limits/gains, 0 rad default); edu unchanged
- robonex_data.py: HELD_JOINTS removed (no importer in any repo); UPPER_BODY_JOINTS = model names of
  robonex-common AUXILIARY_JOINTS (IDs 13, 15-18, 20-23), actuated_joints() = loop_closures actuated_joints
  plus UPPER_BODY_JOINTS, filtered to the variant's URDF joints.
- build_mjcf.py: pro 20 / max 21 position actuators and torque sensors; provisional limits applied only to
  joints present in the variant; home keyframe and ctrl use upper_body_default_pos.
- build_isaac_urdf.py: the 9 upper-body joints are revolute with the provisional limits, URDF effort and
  velocity; upper_body_limits_note printed only in pro/max.
- ver2_constants.json: provisional_limits gain the 9 upper-body joints, new upper_body_limits_note and
  upper_body_default_pos (9 x 0.0); every existing value byte-identical (full solve_constants rerun is
  not bit-reproducible, so the keys were added to the committed JSON).
- edu MJCF (4 files) and Isaac URDFs (2 files) rebuilt byte-identical.

PLACEHOLDERS (nothing measured):
- limits: arms +-0.785398 rad, neck pitch +-0.523599 rad (common v1.2.0 AUXILIARY_JOINTS, open item H29)
- gains: arms kp 40 / kv 2, neck kp 20 / kv 1 (common CONTROL_GAINS_BY_JOINT)
- neck dynamics: armature 0, frictionloss 0, default damping (no MOTOR_PHYSICS rs05; RS05 unmeasured)
- default pose: 0 rad on all 9 upper-body joints
Real values: forcerange/effort = URDF = MOTOR_SPECS t_max (rs02 17, rs05 5.5 N m); arm armature rs02 0.0042.
Isaac USDs not regenerated (convert_urdf.py + apply_physical_loops.py pending). Needs robonex-common
>= 1.2.0 (0ccc7f8); requirements.txt still pins v1.1.0.

File: ver2/isaac/max/closed_loop_box/robonex_max_closed_loop_box.urdf (robot description, URDF)
Before this commit: robot robonex_max, 34 links, 33 joints
Joints:
- joint l_elbow_joint: axis (none) -> 0 -1 0; limit (none) -> lower=-0.785398 upper=0.785398 effort=17 velocity=42.9; type fixed -> revolute
- joint l_shoulder_pitch_joint: axis (none) -> 0 -1 0; limit (none) -> lower=-0.785398 upper=0.785398 effort=17 velocity=42.9; type fixed -> revolute
- joint l_shoulder_roll_joint: axis (none) -> -1 0 0; limit (none) -> lower=-0.785398 upper=0.785398 effort=17 velocity=42.9; type fixed -> revolute
- joint l_shoulder_yaw_joint: axis (none) -> 0 0 1; limit (none) -> lower=-0.785398 upper=0.785398 effort=17 velocity=42.9; type fixed -> revolute
- joint neck_pitch_joint: axis (none) -> 0 -1 0; limit (none) -> lower=-0.523599 upper=0.523599 effort=5.5 velocity=50.3; type fixed -> revolute
- joint r_elbow_joint: axis (none) -> 0 1 0; limit (none) -> lower=-0.785398 upper=0.785398 effort=17 velocity=42.9; type fixed -> revolute
- joint r_shoulder_pitch_joint: axis (none) -> 0 1 0; limit (none) -> lower=-0.785398 upper=0.785398 effort=17 velocity=42.9; type fixed -> revolute
- joint r_shoulder_roll_joint: axis (none) -> -1 0 0; limit (none) -> lower=-0.785398 upper=0.785398 effort=17 velocity=42.9; type fixed -> revolute
- joint r_shoulder_yaw_joint: axis (none) -> 0 0 1; limit (none) -> lower=-0.785398 upper=0.785398 effort=17 velocity=42.9; type fixed -> revolute

File: ver2/isaac/max/closed_loop_mesh/robonex_max_closed_loop_mesh.urdf (robot description, URDF)
Before this commit: robot robonex_max, 34 links, 33 joints
Joints:
- joint l_elbow_joint: axis (none) -> 0 -1 0; limit (none) -> lower=-0.785398 upper=0.785398 effort=17 velocity=42.9; type fixed -> revolute
- joint l_shoulder_pitch_joint: axis (none) -> 0 -1 0; limit (none) -> lower=-0.785398 upper=0.785398 effort=17 velocity=42.9; type fixed -> revolute
- joint l_shoulder_roll_joint: axis (none) -> -1 0 0; limit (none) -> lower=-0.785398 upper=0.785398 effort=17 velocity=42.9; type fixed -> revolute
- joint l_shoulder_yaw_joint: axis (none) -> 0 0 1; limit (none) -> lower=-0.785398 upper=0.785398 effort=17 velocity=42.9; type fixed -> revolute
- joint neck_pitch_joint: axis (none) -> 0 -1 0; limit (none) -> lower=-0.523599 upper=0.523599 effort=5.5 velocity=50.3; type fixed -> revolute
- joint r_elbow_joint: axis (none) -> 0 1 0; limit (none) -> lower=-0.785398 upper=0.785398 effort=17 velocity=42.9; type fixed -> revolute
- joint r_shoulder_pitch_joint: axis (none) -> 0 1 0; limit (none) -> lower=-0.785398 upper=0.785398 effort=17 velocity=42.9; type fixed -> revolute
- joint r_shoulder_roll_joint: axis (none) -> -1 0 0; limit (none) -> lower=-0.785398 upper=0.785398 effort=17 velocity=42.9; type fixed -> revolute
- joint r_shoulder_yaw_joint: axis (none) -> 0 0 1; limit (none) -> lower=-0.785398 upper=0.785398 effort=17 velocity=42.9; type fixed -> revolute

File: ver2/isaac/pro/closed_loop_box/robonex_pro_closed_loop_box.urdf (robot description, URDF)
Before this commit: robot robonex_pro, 33 links, 32 joints
Joints:
- joint l_elbow_joint: axis (none) -> 0 -1 0; limit (none) -> lower=-0.785398 upper=0.785398 effort=17 velocity=42.9; type fixed -> revolute
- joint l_shoulder_pitch_joint: axis (none) -> 0 -1 0; limit (none) -> lower=-0.785398 upper=0.785398 effort=17 velocity=42.9; type fixed -> revolute
- joint l_shoulder_roll_joint: axis (none) -> -1 0 0; limit (none) -> lower=-0.785398 upper=0.785398 effort=17 velocity=42.9; type fixed -> revolute
- joint l_shoulder_yaw_joint: axis (none) -> 0 0 1; limit (none) -> lower=-0.785398 upper=0.785398 effort=17 velocity=42.9; type fixed -> revolute
- joint r_elbow_joint: axis (none) -> 0 1 0; limit (none) -> lower=-0.785398 upper=0.785398 effort=17 velocity=42.9; type fixed -> revolute
- joint r_shoulder_pitch_joint: axis (none) -> 0 1 0; limit (none) -> lower=-0.785398 upper=0.785398 effort=17 velocity=42.9; type fixed -> revolute
- joint r_shoulder_roll_joint: axis (none) -> -1 0 0; limit (none) -> lower=-0.785398 upper=0.785398 effort=17 velocity=42.9; type fixed -> revolute
- joint r_shoulder_yaw_joint: axis (none) -> 0 0 1; limit (none) -> lower=-0.785398 upper=0.785398 effort=17 velocity=42.9; type fixed -> revolute

File: ver2/isaac/pro/closed_loop_mesh/robonex_pro_closed_loop_mesh.urdf (robot description, URDF)
Before this commit: robot robonex_pro, 33 links, 32 joints
Joints:
- joint l_elbow_joint: axis (none) -> 0 -1 0; limit (none) -> lower=-0.785398 upper=0.785398 effort=17 velocity=42.9; type fixed -> revolute
- joint l_shoulder_pitch_joint: axis (none) -> 0 -1 0; limit (none) -> lower=-0.785398 upper=0.785398 effort=17 velocity=42.9; type fixed -> revolute
- joint l_shoulder_roll_joint: axis (none) -> -1 0 0; limit (none) -> lower=-0.785398 upper=0.785398 effort=17 velocity=42.9; type fixed -> revolute
- joint l_shoulder_yaw_joint: axis (none) -> 0 0 1; limit (none) -> lower=-0.785398 upper=0.785398 effort=17 velocity=42.9; type fixed -> revolute
- joint r_elbow_joint: axis (none) -> 0 1 0; limit (none) -> lower=-0.785398 upper=0.785398 effort=17 velocity=42.9; type fixed -> revolute
- joint r_shoulder_pitch_joint: axis (none) -> 0 1 0; limit (none) -> lower=-0.785398 upper=0.785398 effort=17 velocity=42.9; type fixed -> revolute
- joint r_shoulder_roll_joint: axis (none) -> -1 0 0; limit (none) -> lower=-0.785398 upper=0.785398 effort=17 velocity=42.9; type fixed -> revolute
- joint r_shoulder_yaw_joint: axis (none) -> 0 0 1; limit (none) -> lower=-0.785398 upper=0.785398 effort=17 velocity=42.9; type fixed -> revolute

Commit message: [Edit] Regenerate pro/max URDF/MJCF and constants for the common v1.2.0 limits (neck pitch ±73°, shoulder pitch ±100°); edu unchanged

File: ver2/isaac/max/closed_loop_box/robonex_max_closed_loop_box.urdf (robot description, URDF)
Before this commit: robot robonex_max, 34 links, 33 joints
Joints:
- joint l_shoulder_pitch_joint: limit lower=-0.785398 upper=0.785398 effort=17 velocity=42.9 -> lower=-1.745329 upper=1.745329 effort=17 velocity=42.9
- joint neck_pitch_joint: limit lower=-0.523599 upper=0.523599 effort=5.5 velocity=50.3 -> lower=-1.274090 upper=1.274090 effort=5.5 velocity=50.3
- joint r_shoulder_pitch_joint: limit lower=-0.785398 upper=0.785398 effort=17 velocity=42.9 -> lower=-1.745329 upper=1.745329 effort=17 velocity=42.9

File: ver2/isaac/max/closed_loop_mesh/robonex_max_closed_loop_mesh.urdf (robot description, URDF)
Before this commit: robot robonex_max, 34 links, 33 joints
Joints:
- joint l_shoulder_pitch_joint: limit lower=-0.785398 upper=0.785398 effort=17 velocity=42.9 -> lower=-1.745329 upper=1.745329 effort=17 velocity=42.9
- joint neck_pitch_joint: limit lower=-0.523599 upper=0.523599 effort=5.5 velocity=50.3 -> lower=-1.274090 upper=1.274090 effort=5.5 velocity=50.3
- joint r_shoulder_pitch_joint: limit lower=-0.785398 upper=0.785398 effort=17 velocity=42.9 -> lower=-1.745329 upper=1.745329 effort=17 velocity=42.9

File: ver2/isaac/pro/closed_loop_box/robonex_pro_closed_loop_box.urdf (robot description, URDF)
Before this commit: robot robonex_pro, 33 links, 32 joints
Joints:
- joint l_shoulder_pitch_joint: limit lower=-0.785398 upper=0.785398 effort=17 velocity=42.9 -> lower=-1.745329 upper=1.745329 effort=17 velocity=42.9
- joint r_shoulder_pitch_joint: limit lower=-0.785398 upper=0.785398 effort=17 velocity=42.9 -> lower=-1.745329 upper=1.745329 effort=17 velocity=42.9

File: ver2/isaac/pro/closed_loop_mesh/robonex_pro_closed_loop_mesh.urdf (robot description, URDF)
Before this commit: robot robonex_pro, 33 links, 32 joints
Joints:
- joint l_shoulder_pitch_joint: limit lower=-0.785398 upper=0.785398 effort=17 velocity=42.9 -> lower=-1.745329 upper=1.745329 effort=17 velocity=42.9
- joint r_shoulder_pitch_joint: limit lower=-0.785398 upper=0.785398 effort=17 velocity=42.9 -> lower=-1.745329 upper=1.745329 effort=17 velocity=42.9
